File: tinyWASP.kicad_pcb (KiCad board)
At the start: 2 copper layers, 11 x 26 mm, 25 parts, among them J1 ISP, J2 V, J3 G, J4 BZ, J5 BUZ, J6 B+, J7 B-, Q1 2N7002, SW1 BTN, U1 ATtiny24A-MU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

Commit message: fix: rename library folder and update symbol lib format
Connections:
- net /~CHRG renamed /~{CHRG}
Other:
- net class Default removed
